Commit message: Add online state-field training and safe batched planning

File: src/ur_mntfields_arm_sim/urdf/ur_with_wrist_camera.urdf.xacro (robot description, xacro)
@@ -102,5 +102,6 @@
     <parent link="tool0"/>
     <child link="camera_link"/>
-    <origin xyz="0.0 0.0 0.10" rpy="1.57079632679 -1.57079632679 0"/>
+    <!-- tool -Y is above the wrist; tool +Z remains the viewing direction. -->
+    <origin xyz="0.0 -0.08 0.02" rpy="1.57079632679 -1.57079632679 0"/>
   </joint>
   <link name="camera_color_frame"/>
